Commit message: last updates

File: catkin_ws/src/my_robot/urdf/my_robot.xacro (robot description, xacro)
@@ -183,4 +183,13 @@
     <axis xyz="0 1 0" rpy="0 0 0"/>
   </joint>
+<!-- Camera Optical Joint -->
+  <joint name="camera_optical_joint" type="fixed">
+    <origin xyz="0 0 0" rpy="-1.5707 0 -1.5707"/>
+    <parent link="camera"/>
+    <child link="camera_optical"/>
+  </joint>
+<!-- Camera Optical Link -->
+ <link name="camera_optical">
+  </link>
 <!-- Lidar Sensor -->
   <link name="hokuyo">
